Commit message: update 2026-10-29

File: tractor_description/urdf/drawbar.xacro (robot description, xacro)
@@ -3,5 +3,5 @@
 <xacro:macro name="drawbar" params="idx">
   <!-- Load Vehicle Info from YAML -->
-  <xacro:property name="vehicle_info" value="${load_yaml('$(find tractor_description)/config/vehicle_info.param.yaml')['/**']['ros__parameters']}"/>
+  <xacro:property name="vehicle_info" value="${xacro.load_yaml('$(find tractor_description)/config/vehicle_info.param.yaml')['/**']['ros__parameters']}"/>
   <!-- Extract Parameters -->
   <xacro:property name="trailer_wheel_radius" value="${vehicle_info['trailer_wheel_radius']}"/>

File: tractor_description/urdf/tractor.xacro (robot description, xacro)
@@ -2,5 +2,5 @@
 <robot xmlns:xacro="http://www.ros.org/wiki/xacro" name="tow_tractor">
   <!-- Load Vehicle Info from YAML -->
-  <xacro:property name="vehicle_info" value="${load_yaml('$(find tractor_description)/config/vehicle_info.param.yaml')['/**']['ros__parameters']}"/>
+  <xacro:property name="vehicle_info" value="${xacro.load_yaml('$(find tractor_description)/config/vehicle_info.param.yaml')['/**']['ros__parameters']}"/>
   <!-- Extract Parameters -->
   <xacro:property name="wheel_radius" value="${vehicle_info['wheel_radius']}"/>

File: tractor_description/urdf/tractor_trailer.xacro (robot description, xacro)
@@ -1,4 +1,5 @@
 <?xml version="1.0"?>
 <robot xmlns:xacro="http://www.ros.org/wiki/xacro" name="tractor_trailer">
+  <xacro:arg name="num_trailers" default="$(optenv NUM_TRAILERS 4)"/>
   <!-- Include all individual components -->
   <xacro:include filename="$(find tractor_description)/urdf/tractor.xacro" />
@@ -8,10 +9,12 @@
   <xacro:drawbar idx="1"/>
   <xacro:trailer idx="1"/>
-  <xacro:drawbar idx="2"/>
-  <xacro:trailer idx="2"/>
-  <xacro:drawbar idx="3"/>
-  <xacro:trailer idx="3"/>
-  <xacro:drawbar idx="4"/>
-  <xacro:trailer idx="4"/>
+  <xacro:if value="${'$(arg num_trailers)' == '4'}">
+    <xacro:drawbar idx="2"/>
+    <xacro:trailer idx="2"/>
+    <xacro:drawbar idx="3"/>
+    <xacro:trailer idx="3"/>
+    <xacro:drawbar idx="4"/>
+    <xacro:trailer idx="4"/>
+  </xacro:if>
   <!-- Set 1 -->
   <joint name="tractor_to_drawbar_1" type="floating">
@@ -26,35 +29,37 @@
   </joint>
   <!-- Set 2 -->
-  <joint name="trailer_to_drawbar_2" type="floating">
-    <parent link="trailer_rear_hitch_link_1"/>
-    <child link="drawbar_hitch_link_2"/>
-    <origin xyz="0 0 0" rpy="0 0 0"/>
-  </joint>
-  <joint name="drawbar_to_trailer_2" type="floating">
-    <parent link="drawbar_top_hitch_link_2"/>
-    <child link="trailer_front_hitch_link_2"/>
-    <origin xyz="0 0 0" rpy="0 0 0"/>
-  </joint>
-  <!-- Set 3 -->
-  <joint name="trailer_to_drawbar_3" type="floating">
-    <parent link="trailer_rear_hitch_link_2"/>
-    <child link="drawbar_hitch_link_3"/>
-    <origin xyz="0 0 0" rpy="0 0 0"/>
-  </joint>
-  <joint name="drawbar_to_trailer_3" type="floating">
-    <parent link="drawbar_top_hitch_link_3"/>
-    <child link="trailer_front_hitch_link_3"/>
-    <origin xyz="0 0 0" rpy="0 0 0"/>
-  </joint>
-  <!-- Set 4 -->
-  <joint name="trailer_to_drawbar_4" type="floating">
-    <parent link="trailer_rear_hitch_link_3"/>
-    <child link="drawbar_hitch_link_4"/>
-    <origin xyz="0 0 0" rpy="0 0 0"/>
-  </joint>
-  <joint name="drawbar_to_trailer_4" type="floating">
-    <parent link="drawbar_top_hitch_link_4"/>
-    <child link="trailer_front_hitch_link_4"/>
-    <origin xyz="0 0 0" rpy="0 0 0"/>
-  </joint>
+  <xacro:if value="${'$(arg num_trailers)' == '4'}">
+    <joint name="trailer_to_drawbar_2" type="floating">
+      <parent link="trailer_rear_hitch_link_1"/>
+      <child link="drawbar_hitch_link_2"/>
+      <origin xyz="0 0 0" rpy="0 0 0"/>
+    </joint>
+    <joint name="drawbar_to_trailer_2" type="floating">
+      <parent link="drawbar_top_hitch_link_2"/>
+      <child link="trailer_front_hitch_link_2"/>
+      <origin xyz="0 0 0" rpy="0 0 0"/>
+    </joint>
+    <!-- Set 3 -->
+    <joint name="trailer_to_drawbar_3" type="floating">
+      <parent link="trailer_rear_hitch_link_2"/>
+      <child link="drawbar_hitch_link_3"/>
+      <origin xyz="0 0 0" rpy="0 0 0"/>
+    </joint>
+    <joint name="drawbar_to_trailer_3" type="floating">
+      <parent link="drawbar_top_hitch_link_3"/>
+      <child link="trailer_front_hitch_link_3"/>
+      <origin xyz="0 0 0" rpy="0 0 0"/>
+    </joint>
+    <!-- Set 4 -->
+    <joint name="trailer_to_drawbar_4" type="floating">
+      <parent link="trailer_rear_hitch_link_3"/>
+      <child link="drawbar_hitch_link_4"/>
+      <origin xyz="0 0 0" rpy="0 0 0"/>
+    </joint>
+    <joint name="drawbar_to_trailer_4" type="floating">
+      <parent link="drawbar_top_hitch_link_4"/>
+      <child link="trailer_front_hitch_link_4"/>
+      <origin xyz="0 0 0" rpy="0 0 0"/>
+    </joint>
+  </xacro:if>
 </robot>

File: tractor_description/urdf/trailer.xacro (robot description, xacro)
@@ -3,5 +3,5 @@
 <xacro:macro name="trailer" params="idx">
   <!-- Load Vehicle Info from YAML -->
-  <xacro:property name="vehicle_info" value="${load_yaml('$(find tractor_description)/config/vehicle_info.param.yaml')['/**']['ros__parameters']}"/>
+  <xacro:property name="vehicle_info" value="${xacro.load_yaml('$(find tractor_description)/config/vehicle_info.param.yaml')['/**']['ros__parameters']}"/>
   <!-- Extract Parameters -->
   <xacro:property name="trailer_wheel_radius" value="${vehicle_info['trailer_wheel_radius']}"/>

File: tractor_sensor_kit_description/urdf/sensor_kit.xacro (robot description, xacro)
@@ -57,4 +57,28 @@
       <origin xyz="0.0 0.0 0.2" rpy="0 0 0"/>
     </joint>
+    <!-- Drawbar IMU (Center of drawbar, 0.2m high) -->
+    <link name="drawbar_imu_link">
+      <visual>
+        <geometry><box size="0.1 0.1 0.05"/></geometry>
+        <material name="drawbar_imu_mat"><color rgba="0.0 0.8 0.0 1.0"/></material>
+      </visual>
+    </link>
+    <joint name="drawbar_imu_joint" type="fixed">
+      <parent link="drawbar_link_1"/>
+      <child link="drawbar_imu_link"/>
+      <origin xyz="0.0 0.0 0.2" rpy="0 0 0"/>
+    </joint>
+    <!-- Trailer IMU (Center of trailer, 0.2m high) -->
+    <link name="trailer_imu_link">
+      <visual>
+        <geometry><box size="0.1 0.1 0.05"/></geometry>
+        <material name="trailer_imu_mat"><color rgba="0.0 0.8 0.0 1.0"/></material>
+      </visual>
+    </link>
+    <joint name="trailer_imu_joint" type="fixed">
+      <parent link="trailer_link_1"/>
+      <child link="trailer_imu_link"/>
+      <origin xyz="0.0 0.0 0.2" rpy="0 0 0"/>
+    </joint>
   </xacro:macro>
 </robot>
